File: kp-ptr/IO.kicad_sch (KiCad schematic)
At the start: 10 parts, among them Q5 NMOS_SOT23

Commit message: Footprinty drobnicy
Signed-off-by: kretu <krecik@gmail.com>
Parts:
- D5: footprint Diode_THT:D_DO-35_SOD27_P7.62mm_Horizontal -> Diode_SMD:D_SOD-123
- R40: footprint Resistor_SMD:R_01005_0402Metric_Pad0.57x0.30mm_HandSolder -> Resistor_SMD:R_0402_1005Metric_Pad0.72x0.64mm_HandSolder
Changed lines of the file:
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@@
       (effects (font (size 1.27 1.27)) (justify left))
     )
-    (property "Footprint" "Diode_THT:D_DO-35_SOD27_P7.62mm_Horizontal" (id 2) (at 45.085 95.25 0)
+    (property "Footprint" "Diode_SMD:D_SOD-123" (id 2) (at 45.085 95.25 0)
       (effects (font (size 1.27 1.27)) hide)
     )
@@
     (property "Reference" "R40" (id 0) (at 45.72 69.85 90))
     (property "Value" "1k" (id 1) (at 45.72 74.93 90))
-    (property "Footprint" "Resistor_SMD:R_01005_0402Metric_Pad0.57x0.30mm_HandSolder" (id 2) (at 46.99 70.612 90)
+    (property "Footprint" "Resistor_SMD:R_0402_1005Metric_Pad0.72x0.64mm_HandSolder" (id 2) (at 46.99 70.612 90)
       (effects (font (size 1.27 1.27)) hide)
     )

Commit message: Szlifowanie schematu
Parts:
- removed D6, D8: LED, LED_SMD:LED_0402_1005Metric_Pad0.77x0.64mm_HandSolder, symbol Device:LED
- removed R40: 1k, Resistor_SMD:R_0402_1005Metric_Pad0.72x0.64mm_HandSolder, symbol Device:R
- added D? (x3): WS2812B-2020, symbol KP-PTR_lib:WS2812B-2020
- added D?: LED, LED_SMD:LED_0402_1005Metric_Pad0.77x0.64mm_HandSolder, symbol Device:LED
- added R? (x6): 1k, Resistor_SMD:R_0402_1005Metric_Pad0.72x0.64mm_HandSolder, symbol Device:R
- added R?: 10k, Resistor_SMD:R_0402_1005Metric_Pad0.72x0.64mm_HandSolder, symbol Device:R
Connections:
- net +3V3: now also D?.4 (VDD), D?.4 (VDD), D?.4 (VDD)
- net Earth: now also D?.1 (K), D?.2 (GND), D?.2 (GND), D?.2 (GND), R?.2
- net at R38.1: now also D?.3 (DIN)
- new net: D?.1 (DOUT), D?.3 (DIN) (x2)
- new net: D?.2 (A), R?.1
- new net: R?.1, R?.1
- new net SERVO_1: R?.2
- new net SERVO_2: R?.2
- new net SERVO_3: R?.2
- new net SERVO_4: R?.2
- new net SERVO_EN: R?.2, R?.2
- no-connect marks 0 -> 1
Other:
- moved on the sheet: D7, R38, R39

Commit message: Update po spotkaniu
Parts:
- added C48, C49, C50: 100nF, Capacitor_SMD:C_0402_1005Metric, symbol Device:C
- added J10: Conn_01x10_Male, Connector_JST:JST_GH_BM10B-GHS-TBT_1x10-1MP_P1.25mm_Vertical, symbol Connector:Conn_01x10_Male
- added J12, J5: Conn_01x06_Male, Connector_JST:JST_GH_BM06B-GHS-TBT_1x06-1MP_P1.25mm_Vertical, symbol Connector:Conn_01x06_Male
- added J13: Conn_01x02_Male, TerminalBlock_TE-Connectivity:TerminalBlock_TE_282834-2_1x02_P2.54mm_Horizontal, symbol Connector:Conn_01x02_Male
- D12: renamed from D?; footprint LED_SMD:LED_0402_1005Metric_Pad0.77x0.64mm_HandSolder -> LED_SMD:LED_0603_1608Metric
- D7: footprint LED_SMD:LED_0402_1005Metric_Pad0.77x0.64mm_HandSolder -> LED_SMD:LED_0603_1608Metric
- LS1: footprint KP-PTR_lib:BUZZER CBT-09 -> Buzzer_Beeper:Buzzer_12x9.5RM7.6
- R34, R35, R36, R40, R61, R62, R63: renamed from R?; footprint Resistor_SMD:R_0402_1005Metric_Pad0.72x0.64mm_HandSolder -> Resistor_SMD:R_0402_1005Metric
- R37, R38, R39: footprint Resistor_SMD:R_0402_1005Metric_Pad0.72x0.64mm_HandSolder -> Resistor_SMD:R_0402_1005Metric
- gave numbers to parts that had none: 3
Connections:
- net +3V3: now also C48.1, C49.1, C50.1
- net +5V: now also J10.1 (Pin_1), J12.1 (Pin_1), J5.1 (Pin_1)
- net Earth: now also C48.2, C49.2, C50.2, J10.10 (Pin_10), J10.9 (Pin_9), J12.6 (Pin_6), J13.2 (Pin_2), J5.6 (Pin_6)
- net I2C_SCL: now also J12.4 (Pin_4), J5.4 (Pin_4)
- net I2C_SDA: now also J12.5 (Pin_5), J5.5 (Pin_5)
- net UART1_IN: now also J10.3 (Pin_3), J12.3 (Pin_3), J5.3 (Pin_3)
- net UART1_OUT: now also J10.2 (Pin_2), J12.2 (Pin_2), J5.2 (Pin_2)
- net at R35.1: now also J10.4 (Pin_4)
- net at R61.1: now also J10.7 (Pin_7)
- net at R36.1: now also J10.5 (Pin_5)
- net at R62.1, R63.1: now also J10.8 (Pin_8)
- net at R40.1: now also J10.6 (Pin_6)
- new net VCC: J13.1 (Pin_1)
Other:
- moved on the sheet: D12, R34, R62, R63
