File: kp-ptr/IO.kicad_sch (KiCad schematic)
At the start: 25 parts, among them J10 Conn_01x10_Male, J12 Conn_01x06_Male, J13 Conn_01x02_Male, J5 Conn_01x06_Male, Q5 NMOS_SOT23

Commit message: Grupowanie
Parts:
- renumbered C48 to C44, C49 to C45, C50 to C46, D12 to D10, D5 to D11, D7 to D12, J5 to J6, J10 to J7, J12 to J8, J13 to J9, Q5 to Q1, R40 to R37, R61 to R38, R62 to R39, R38 to R40, R39 to R41, R37 to R42, R63 to R43
Connections:
- net +3V3: now also LS1.1 (+); no longer LS1.P
- net at D11.2 (A), Q1.3 (D): now also LS1.2 (-); no longer LS1.M

Commit message: 1 próba pomieszczenia wszystkiego
Signed-off-by: kretu <krecik@gmail.com>
Parts:
- J9: footprint TerminalBlock_TE-Connectivity:TerminalBlock_TE_282834-2_1x02_P2.54mm_Horizontal -> Connector_JST:JST_GH_BM02B-GHS-TBT_1x02-1MP_P1.25mm_Vertical
Changed lines of the file:
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@@
       (effects (font (size 1.27 1.27)) (justify right))
     )
-    (property "Footprint" "TerminalBlock_TE-Connectivity:TerminalBlock_TE_282834-2_1x02_P2.54mm_Horizontal" (id 2) (at 143.51 182.245 0)
+    (property "Footprint" "Connector_JST:JST_GH_BM02B-GHS-TBT_1x02-1MP_P1.25mm_Vertical" (id 2) (at 143.51 182.245 0)
       (effects (font (size 1.27 1.27)) hide)
     )

Commit message: swiatelko w tunelu aby zmiescic wszystko
Parts:
- J9: footprint Connector_JST:JST_GH_BM02B-GHS-TBT_1x02-1MP_P1.25mm_Vertical -> TerminalBlock_TE-Connectivity:TerminalBlock_TE_282834-2_1x02_P2.54mm_Horizontal
Changed lines of the file:
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@@
       (effects (font (size 1.27 1.27)) (justify right))
     )
-    (property "Footprint" "Connector_JST:JST_GH_BM02B-GHS-TBT_1x02-1MP_P1.25mm_Vertical" (id 2) (at 143.51 182.245 0)
+    (property "Footprint" "TerminalBlock_TE-Connectivity:TerminalBlock_TE_282834-2_1x02_P2.54mm_Horizontal" (id 2) (at 143.51 182.245 0)
       (effects (font (size 1.27 1.27)) hide)
     )

Commit message: chyba wszystkie footprinty
Parts:
- D13, D14, D15: footprint (none) -> KP-PTR_lib:WS2812B-2020
Changed lines of the file:
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@@
   (symbol (lib_id "power:VCC") (at 138.43 182.245 0) (unit 1)
     (in_bom yes) (on_board yes)
-    (property "Reference" "#PWR0157" (id 0) (at 138.43 186.055 0)
+    (property "Reference" "#PWR0158" (id 0) (at 138.43 186.055 0)
       (effects (font (size 1.27 1.27)) hide)
     )
@@
   (symbol (lib_id "power:Earth") (at 83.82 190.5 0) (unit 1)
     (in_bom yes) (on_board yes) (fields_autoplaced)
-    (property "Reference" "#PWR0148" (id 0) (at 83.82 196.85 0)
+    (property "Reference" "#PWR0149" (id 0) (at 83.82 196.85 0)
       (effects (font (size 1.27 1.27)) hide)
     )
@@
   (symbol (lib_id "power:+3.3V") (at 108.585 21.59 0) (unit 1)
     (in_bom yes) (on_board yes)
-    (property "Reference" "#PWR0149" (id 0) (at 108.585 25.4 0)
+    (property "Reference" "#PWR0150" (id 0) (at 108.585 25.4 0)
       (effects (font (size 1.27 1.27)) hide)
     )
@@
   (symbol (lib_id "power:Earth") (at 71.12 46.99 90) (unit 1)
     (in_bom yes) (on_board yes) (fields_autoplaced)
-    (property "Reference" "#PWR0142" (id 0) (at 77.47 46.99 0)
+    (property "Reference" "#PWR0143" (id 0) (at 77.47 46.99 0)
       (effects (font (size 1.27 1.27)) hide)
     )
@@
   (symbol (lib_id "power:Earth") (at 40.005 190.5 0) (unit 1)
     (in_bom yes) (on_board yes) (fields_autoplaced)
-    (property "Reference" "#PWR0135" (id 0) (at 40.005 196.85 0)
+    (property "Reference" "#PWR0136" (id 0) (at 40.005 196.85 0)
       (effects (font (size 1.27 1.27)) hide)
     )
@@
   (symbol (lib_id "power:+5V") (at 83.185 177.8 0) (unit 1)
     (in_bom yes) (on_board yes)
-    (property "Reference" "#PWR0145" (id 0) (at 83.185 181.61 0)
+    (property "Reference" "#PWR0146" (id 0) (at 83.185 181.61 0)
       (effects (font (size 1.27 1.27)) hide)
     )
@@
   (symbol (lib_id "power:+3.3V") (at 83.82 49.53 0) (unit 1)
     (in_bom yes) (on_board yes)
-    (property "Reference" "#PWR0146" (id 0) (at 83.82 53.34 0)
+    (property "Reference" "#PWR0147" (id 0) (at 83.82 53.34 0)
       (effects (font (size 1.27 1.27)) hide)
     )
@@
   (symbol (lib_id "power:Earth") (at 133.35 36.83 0) (unit 1)
     (in_bom yes) (on_board yes) (fields_autoplaced)
-    (property "Reference" "#PWR0154" (id 0) (at 133.35 43.18 0)
+    (property "Reference" "#PWR0155" (id 0) (at 133.35 43.18 0)
       (effects (font (size 1.27 1.27)) hide)
     )
@@
     (property "Reference" "D14" (id 0) (at 111.76 22.86 0))
     (property "Value" "WS2812B-2020" (id 1) (at 108.585 41.275 0))
-    (property "Footprint" "" (id 2) (at 109.855 36.83 0)
+    (property "Footprint" "KP-PTR_lib:WS2812B-2020" (id 2) (at 109.855 36.83 0)
       (effects (font (size 1.27 1.27)) (justify left top) hide)
     )
@@
   (symbol (lib_id "power:+3.3V") (at 133.35 21.59 0) (unit 1)
     (in_bom yes) (on_board yes)
-    (property "Reference" "#PWR0153" (id 0) (at 133.35 25.4 0)
+    (property "Reference" "#PWR0154" (id 0) (at 133.35 25.4 0)
       (effects (font (size 1.27 1.27)) hide)
     )
@@
   (symbol (lib_id "power:+3.3V") (at 55.88 87.63 0) (unit 1)
     (in_bom yes) (on_board yes)
-    (property "Reference" "#PWR0137" (id 0) (at 55.88 91.44 0)
+    (property "Reference" "#PWR0138" (id 0) (at 55.88 91.44 0)
       (effects (font (size 1.27 1.27)) hide)
     )
@@
   (symbol (lib_id "power:+5V") (at 59.69 131.445 0) (unit 1)
     (in_bom yes) (on_board yes)
-    (property "Reference" "#PWR0139" (id 0) (at 59.69 135.255 0)
+    (property "Reference" "#PWR0140" (id 0) (at 59.69 135.255 0)
       (effects (font (size 1.27 1.27)) hide)
     )
@@
   (symbol (lib_id "power:Earth") (at 109.22 57.785 0) (unit 1)
     (in_bom yes) (on_board yes) (fields_autoplaced)
-    (property "Reference" "#PWR0152" (id 0) (at 109.22 64.135 0)
+    (property "Reference" "#PWR0153" (id 0) (at 109.22 64.135 0)
       (effects (font (size 1.27 1.27)) hide)
     )
@@
   (symbol (lib_id "power:Earth") (at 133.35 57.15 0) (unit 1)
     (in_bom yes) (on_board yes) (fields_autoplaced)
-    (property "Reference" "#PWR0156" (id 0) (at 133.35 63.5 0)
+    (property "Reference" "#PWR0157" (id 0) (at 133.35 63.5 0)
       (effects (font (size 1.27 1.27)) hide)
     )
@@
     (property "Reference" "D15" (id 0) (at 136.525 22.86 0))
     (property "Value" "WS2812B-2020" (id 1) (at 133.35 41.275 0))
-    (property "Footprint" "" (id 2) (at 134.62 36.83 0)
+    (property "Footprint" "KP-PTR_lib:WS2812B-2020" (id 2) (at 134.62 36.83 0)
       (effects (font (size 1.27 1.27)) (justify left top) hide)
     )
@@
   (symbol (lib_id "power:Earth") (at 59.69 159.385 0) (unit 1)
     (in_bom yes) (on_board yes) (fields_autoplaced)
-    (property "Reference" "#PWR0140" (id 0) (at 59.69 165.735 0)
+    (property "Reference" "#PWR0141" (id 0) (at 59.69 165.735 0)
       (effects (font (size 1.27 1.27)) hide)
     )
@@
   (symbol (lib_id "power:Earth") (at 83.185 36.83 0) (unit 1)
     (in_bom yes) (on_board yes) (fields_autoplaced)
-    (property "Reference" "#PWR0144" (id 0) (at 83.185 43.18 0)
+    (property "Reference" "#PWR0145" (id 0) (at 83.185 43.18 0)
       (effects (font (size 1.27 1.27)) hide)
     )
@@
   (symbol (lib_id "power:+3.3V") (at 133.35 49.53 0) (unit 1)
     (in_bom yes) (on_board yes)
-    (property "Reference" "#PWR0155" (id 0) (at 133.35 53.34 0)
+    (property "Reference" "#PWR0156" (id 0) (at 133.35 53.34 0)
       (effects (font (size 1.27 1.27)) hide)
     )
@@
   (symbol (lib_id "power:Earth") (at 55.88 115.57 0) (unit 1)
     (in_bom yes) (on_board yes) (fields_autoplaced)
-    (property "Reference" "#PWR0138" (id 0) (at 55.88 121.92 0)
+    (property "Reference" "#PWR0139" (id 0) (at 55.88 121.92 0)
       (effects (font (size 1.27 1.27)) hide)
     )
@@
   (symbol (lib_id "power:Earth") (at 83.82 57.15 0) (unit 1)
     (in_bom yes) (on_board yes) (fields_autoplaced)
-    (property "Reference" "#PWR0147" (id 0) (at 83.82 63.5 0)
+    (property "Reference" "#PWR0148" (id 0) (at 83.82 63.5 0)
       (effects (font (size 1.27 1.27)) hide)
     )
@@
   (symbol (lib_id "power:Earth") (at 66.04 159.385 0) (unit 1)
     (in_bom yes) (on_board yes) (fields_autoplaced)
-    (property "Reference" "#PWR0141" (id 0) (at 66.04 165.735 0)
+    (property "Reference" "#PWR0142" (id 0) (at 66.04 165.735 0)
       (effects (font (size 1.27 1.27)) hide)
     )
@@
   (symbol (lib_id "power:+3.3V") (at 109.22 50.165 0) (unit 1)
     (in_bom yes) (on_board yes)
-    (property "Reference" "#PWR0151" (id 0) (at 109.22 53.975 0)
+    (property "Reference" "#PWR0152" (id 0) (at 109.22 53.975 0)
       (effects (font (size 1.27 1.27)) hide)
     )
@@
   (symbol (lib_id "power:Earth") (at 42.545 164.465 0) (unit 1)
     (in_bom yes) (on_board yes) (fields_autoplaced)
-    (property "Reference" "#PWR0136" (id 0) (at 42.545 170.815 0)
+    (property "Reference" "#PWR0137" (id 0) (at 42.545 170.815 0)
       (effects (font (size 1.27 1.27)) hide)
     )
@@
   (symbol (lib_id "power:+3.3V") (at 83.185 21.59 0) (unit 1)
     (in_bom yes) (on_board yes)
-    (property "Reference" "#PWR0143" (id 0) (at 83.185 25.4 0)
+    (property "Reference" "#PWR0144" (id 0) (at 83.185 25.4 0)
       (effects (font (size 1.27 1.27)) hide)
     )
@@
   (symbol (lib_id "power:+5V") (at 39.37 177.8 0) (unit 1)
     (in_bom yes) (on_board yes)
-    (property "Reference" "#PWR0134" (id 0) (at 39.37 181.61 0)
+    (property "Reference" "#PWR0135" (id 0) (at 39.37 181.61 0)
       (effects (font (size 1.27 1.27)) hide)
     )
@@
   (symbol (lib_id "power:Earth") (at 108.585 36.83 0) (unit 1)
     (in_bom yes) (on_board yes) (fields_autoplaced)
-    (property "Reference" "#PWR0150" (id 0) (at 108.585 43.18 0)
+    (property "Reference" "#PWR0151" (id 0) (at 108.585 43.18 0)
       (effects (font (size 1.27 1.27)) hide)
     )
@@
     (property "Reference" "D13" (id 0) (at 86.36 22.86 0))
     (property "Value" "WS2812B-2020" (id 1) (at 83.185 41.275 0))
-    (property "Footprint" "" (id 2) (at 84.455 36.83 0)
+    (property "Footprint" "KP-PTR_lib:WS2812B-2020" (id 2) (at 84.455 36.83 0)
       (effects (font (size 1.27 1.27)) (justify left top) hide)
     )
@@
   (symbol (lib_id "power:Earth") (at 138.43 184.785 0) (unit 1)
     (in_bom yes) (on_board yes) (fields_autoplaced)
-    (property "Reference" "#PWR0158" (id 0) (at 138.43 191.135 0)
-      (effects (font (size 1.27 1.27)) hide)
-    )
+    (property "Reference" "#PWR0159" (id 0) (at 138.43 191.135 0)
+      (effects (font (size 1.27 1.27)) hide)
+    )

Commit message: PCB update
Parts:
- added R27, R32: 10k, Resistor_SMD:R_0402_1005Metric, symbol Device:R
Connections:
- net +3V3: now also R27.2, R32.2
- net I2C_SCL: now also R27.1
- net I2C_SDA: now also R32.1
Other:
- note added: "Servo power supply"
Changed lines of the file:
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@@
+    (stroke (width 0) (type default) (color 0 0 0 0))
+  )
+  (wire (pts (xy 105.41 158.75) (xy 105.41 162.56))
     (stroke (width 0) (type default) (color 0 0 0 0))
   )
@@
     (stroke (width 0) (type default) (color 0 0 0 0))
   )
+  (wire (pts (xy 100.965 165.1) (xy 113.03 165.1))
+    (stroke (width 0) (type default) (color 0 0 0 0))
+  )
   (wire (pts (xy 52.705 144.145) (xy 66.04 144.145))
     (stroke (width 0) (type default) (color 0 0 0 0))
@@
     (stroke (width 0) (type default) (color 0 0 0 0))
   )
+  (wire (pts (xy 105.41 162.56) (xy 100.965 162.56))
+    (stroke (width 0) (type default) (color 0 0 0 0))
+  )
   (wire (pts (xy 59.69 151.765) (xy 59.69 149.225))
     (stroke (width 0) (type default) (color 0 0 0 0))
@@
     (stroke (width 0) (type default) (color 0 0 0 0))
   )
+  (wire (pts (xy 113.03 165.1) (xy 113.03 158.75))
+    (stroke (width 0) (type default) (color 0 0 0 0))
+  )
+  (text "Servo power supply" (at 135.89 191.77 0)
+    (effects (font (size 1.27 1.27)) (justify left bottom))
+  )
   (global_label "UART1_OUT" (shape input) (at 82.55 180.34 180) (fields_autoplaced)
     (effects (font (size 1.27 1.27)) (justify right))
@@
     )
   )
+  (global_label "I2C_SCL" (shape input) (at 100.965 162.56 180) (fields_autoplaced)
+    (effects (font (size 1.27 1.27)) (justify right))
+    (property "Intersheet References" "${INTERSHEET_REFS}" (id 0) (at 90.9924 162.4806 0)
+      (effects (font (size 1.27 1.27)) (justify right) hide)
+    )
+  )
   (global_label "SERVO_2" (shape input) (at 36.83 141.605 180) (fields_autoplaced)
     (effects (font (size 1.27 1.27)) (justify right))
@@
     (effects (font (size 1.27 1.27)) (justify right))
     (property "Intersheet References" "${INTERSHEET_REFS}" (id 0) (at 24.9221 149.1456 0)
+      (effects (font (size 1.27 1.27)) (justify right) hide)
+    )
+  )
+  (global_label "I2C_SDA" (shape input) (at 100.965 165.1 180) (fields_autoplaced)
+    (effects (font (size 1.27 1.27)) (justify right))
+    (property "Intersheet References" "${INTERSHEET_REFS}" (id 0) (at 90.9319 165.0206 0)
       (effects (font (size 1.27 1.27)) (justify right) hide)
     )
@@
     (property "PRICE" "None" (id 9) (at 55.88 95.25 0)
       (effects (font (size 1.27 1.27)) (justify left bottom) hide)
+    )
+    (pin "1")
+    (pin "2")
+  )
+  (symbol (lib_id "Device:R") (at 105.41 154.94 180) (unit 1)
+    (in_bom yes) (on_board yes)
+    (property "Reference" "R27" (id 0) (at 107.95 153.67 90))
+    (property "Value" "10k" (id 1) (at 102.87 153.67 90))
+    (property "Footprint" "Resistor_SMD:R_0402_1005Metric" (id 2) (at 107.188 154.94 90)
+      (effects (font (size 1.27 1.27)) hide)
+    )
+    (property "Datasheet" "~" (id 3) (at 105.41 154.94 0)
+      (effects (font (size 1.27 1.27)) hide)
     )
     (pin "1")
@@
     (pin "2")
   )
+  (symbol (lib_id "Device:R") (at 113.03 154.94 180) (unit 1)
+    (in_bom yes) (on_board yes)
+    (property "Reference" "R32" (id 0) (at 115.57 153.67 90))
+    (property "Value" "10k" (id 1) (at 110.49 153.67 90))
+    (property "Footprint" "Resistor_SMD:R_0402_1005Metric" (id 2) (at 114.808 154.94 90)
+      (effects (font (size 1.27 1.27)) hide)
+    )
+    (property "Datasheet" "~" (id 3) (at 113.03 154.94 0)
+      (effects (font (size 1.27 1.27)) hide)
+    )
+    (pin "1")
+    (pin "2")
+  )
   (symbol (lib_id "Device:R") (at 48.895 146.685 270) (unit 1)
     (in_bom yes) (on_board yes)
@@
     (pin "1")
     (pin "2")
+  )
+  (symbol (lib_id "power:+3.3V") (at 113.03 151.13 0) (unit 1)
+    (in_bom yes) (on_board yes)
+    (property "Reference" "#PWR0176" (id 0) (at 113.03 154.94 0)
+      (effects (font (size 1.27 1.27)) hide)
+    )
+    (property "Value" "+3.3V" (id 1) (at 113.03 147.32 0))
+    (property "Footprint" "" (id 2) (at 113.03 151.13 0)
+      (effects (font (size 1.27 1.27)) hide)
+    )
+    (property "Datasheet" "" (id 3) (at 113.03 151.13 0)
+      (effects (font (size 1.27 1.27)) hide)
+    )
+    (pin "1")
   )
   (symbol (lib_id "power:Earth") (at 133.35 57.15 0) (unit 1)
@@
       (effects (font (size 1.27 1.27)) hide)
     )
+    (pin "1")
+  )
+  (symbol (lib_id "power:+3.3V") (at 105.41 151.13 0) (unit 1)
+    (in_bom yes) (on_board yes)
+    (property "Reference" "#PWR0133" (id 0) (at 105.41 154.94 0)
+      (effects (font (size 1.27 1.27)) hide)
+    )
+    (property "Value" "+3.3V" (id 1) (at 105.41 147.32 0))
+    (property "Footprint" "" (id 2) (at 105.41 151.13 0)
+      (effects (font (size 1.27 1.27)) hide)
+    )
+    (property "Datasheet" "" (id 3) (at 105.41 151.13 0)
+      (effects (font (size 1.27 1.27)) hide)
+    )
