File: kp-ptr/IO.kicad_sch (KiCad schematic)
At the start: 27 parts, among them J6 Conn_01x06_Male, J7 Conn_01x10_Male, J8 Conn_01x06_Male, J9 Conn_01x02_Male, Q1 NMOS_SOT23

Commit message: Parts renumbered! Noice!
Parts:
- renumbered C44 to C51, C46 to C52, C27 to C53, C45 to C54, D13 to D10, D14 to D11, D15 to D12, D12 to D13, D11 to D14, D10 to D15, J7 to J6, J9 to J7, J6 to J8, J8 to J9, R40 to R42, R42 to R43, R35 to R44, R36 to R45, R37 to R46, R38 to R47, R39 to R48, R34 to R49, R27 to R50, R32 to R51, R43 to R52

Commit message: Backup capacitor changed from electro to tantal.
Multiple kung fu changes
Parts:
- added C62, C63, C64, C65: 100nF, Capacitor_SMD:C_0402_1005Metric, symbol Device:C
- added D16, D17, D18, D19: WS2812B-2020, KP-PTR_lib:WS2812B-2020, symbol KP-PTR_lib:WS2812B-2020
Connections:
- net +3V3: now also C62.1, C63.1, C64.1, C65.1, D16.4 (VDD), D17.4 (VDD), D18.4 (VDD), D19.4 (VDD)
- net Earth: now also C62.2, C63.2, C64.2, C65.2, D16.2 (GND), D17.2 (GND), D18.2 (GND), D19.2 (GND)
- net at D13.1 (DOUT): now also D16.3 (DIN)
- new net: D18.1 (DOUT), D19.3 (DIN)
- new net: D17.1 (DOUT), D18.3 (DIN)
- new net: D16.1 (DOUT), D17.3 (DIN)

Commit message: Wersja produkcyjna v1
Parts:
- D15: value LED -> GREEN
Changed lines of the file:
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@@
       (effects (font (size 1.27 1.27)) (justify right))
     )
-    (property "Value" "LED" (id 1) (at 45.72 163.5124 90)
+    (property "Value" "GREEN" (id 1) (at 45.72 163.5124 90)
       (effects (font (size 1.27 1.27)) (justify right))
     )

Commit message: Release v1
Other:
- company: (none) -> Polskie Towarzystwo Rakietowe
- title: (none) -> KP-PTR
- moved on the sheet: D14, D15, J6, J7, J8, J9, LS1, Q1, R43, R44, R45, R46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

Commit message: New schematic revision v1.1:
- added 'DNP' info for few components
- some stylistic improvements
- added comment about I2C pins glitch
Other:
- note added: "LED ARM"
- note added: "LED IGN1"
- note added: "LED IGN2"
- note added: "LED IGN3"
- note added: "LED IGN4"
- note added: "LED READY"
- note added: "LED RX"
- note added: "LED STAT"
- note added: "Servo ext. connector"
- note added: "UART & I2C ext. connectors"
- moved on the sheet: J7, R50, R51
