File: kp-ptr/PSU.kicad_sch (KiCad schematic)
At the start: 17 parts, among them J2 Conn_01x02, J3 Conn_01x02, U8 SPX3819M5-L-3-3

Commit message: Szlifowanie schematu
Parts:
- removed U8: SPX3819M5-L-3-3, Package_TO_SOT_SMD:SOT-23-5, symbol Regulator_Linear:SPX3819M5-L-3-3
- added C?: 10u, Capacitor_SMD:C_0402_1005Metric_Pad0.74x0.62mm_HandSolder, symbol Device:C
- added C?: 1uF, Capacitor_SMD:C_0402_1005Metric_Pad0.74x0.62mm_HandSolder, symbol Device:C
- added D?: G, LED_SMD:LED_0402_1005Metric_Pad0.77x0.64mm_HandSolder, symbol Device:LED
- added F?: 500mA, Fuse:Fuse_1206_3216Metric_Pad1.42x1.75mm_HandSolder, symbol Device:Polyfuse
- added R?: 10k, Resistor_SMD:R_0402_1005Metric_Pad0.72x0.64mm_HandSolder, symbol Device:R
Connections:
- net Earth: now also C?.2, C?.2, R?.2
- net VDD: now also C?.1
- new net: C?.1, F?.2
- new net: D?.1 (K), R?.1
- new net +5V: D?.2 (A), F?.1
Other:
- note added: "Coś na 5V TBD"
- note added: "LDFM33PVR"
- note removed: "Dajemy włącznik czy załączamy podłaczeniem akumulatora? Regulatory napięcia do dobrania. SPXy są sprawdzone w bojach, ale mogą być też inne pinowozgodne"

Commit message: Update po spotkaniu
Parts:
- added U12: LM1117-5.0, symbol Regulator_Linear:LM1117-5.0
- C31: value 1uF -> 10n; footprint Capacitor_SMD:C_0402_1005Metric_Pad0.74x0.62mm_HandSolder -> Capacitor_SMD:C_0402_1005Metric
- C32, C33, C35: footprint Capacitor_SMD:C_0402_1005Metric_Pad0.74x0.62mm_HandSolder -> Capacitor_SMD:C_0402_1005Metric
- C44, C45: renamed from C?; footprint Capacitor_SMD:C_0402_1005Metric_Pad0.74x0.62mm_HandSolder -> Capacitor_SMD:C_0402_1005Metric
- D11: renamed from D?; footprint LED_SMD:LED_0402_1005Metric_Pad0.77x0.64mm_HandSolder -> LED_SMD:LED_0603_1608Metric
- D3, D4: footprint LED_SMD:LED_0402_1005Metric_Pad0.77x0.64mm_HandSolder -> LED_SMD:LED_0603_1608Metric
- F6: renamed from F?; footprint Fuse:Fuse_1206_3216Metric_Pad1.42x1.75mm_HandSolder -> Fuse:Fuse_0805_2012Metric
- R23: renamed from R?; footprint Resistor_SMD:R_0402_1005Metric_Pad0.72x0.64mm_HandSolder -> Resistor_SMD:R_0402_1005Metric
- R24, R25, R26, R27, R29, R30: footprint Resistor_SMD:R_0402_1005Metric_Pad0.72x0.64mm_HandSolder -> Resistor_SMD:R_0402_1005Metric
- gave numbers to parts that had none: 1
Connections:
- net Earth: now also U12.1 (GND)
- net VDD: now also U12.3 (VI)
- net at C45.1, F6.2: now also U12.2 (VO)
Other:
- note removed: "Coś na 5V TBD"
- moved on the sheet: C31, C32, D11, D2, D3, D4, D8, J3, R23, R24, R25, R26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

Commit message: Grupowanie
Parts:
- J2, J3: footprint TerminalBlock_TE-Connectivity:TerminalBlock_TE_282834-2_1x02_P2.54mm_Horizontal -> TerminalBlock_Phoenix:TerminalBlock_Phoenix_MPT-0,5-2-2.54_1x02_P2.54mm_Horizontal
- renumbered C31 to C33, C32 to C34, C33 to C35, C44 to C36, C35 to C37, C45 to C38, D8 to D3, D2 to D4, D3 to D5, D4 to D6, D11 to D7, F6 to F1, R24 to R19, R25 to R20, R26 to R21, R27 to R22, R29 to R23, R30 to R24, R23 to R25, U12 to U8
