File: kp-ptr/igniters.kicad_sch (KiCad schematic)
At the start: 36 parts, among them J10 Conn_01x02, J11 Conn_01x02, J12 Conn_01x02, J13 Conn_01x02, Q2 DMC2025UFDB_v2, Q3 DMC2025UFDB_v2, Q4 DMC2025UFDB_v2, Q5 DMC2025UFDB_v2

Commit message: swiatelko w tunelu aby zmiescic wszystko
Parts:
- J10, J11, J12, J13: footprint TerminalBlock_Phoenix:TerminalBlock_Phoenix_MPT-0,5-2-2.54_1x02_P2.54mm_Horizontal -> TerminalBlock_TE-Connectivity:TerminalBlock_TE_282834-2_1x02_P2.54mm_Horizontal
Changed lines of the file:
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@@
       (effects (font (size 1.27 1.27)) (justify left) hide)
     )
-    (pin "1")
-    (pin "2")
-    (pin "5")
     (pin "3")
     (pin "4")
@@
       (effects (font (size 1.27 1.27)) (justify left) hide)
     )
-    (pin "1")
-    (pin "2")
-    (pin "5")
     (pin "3")
     (pin "4")
@@
       (effects (font (size 1.27 1.27)) (justify left))
     )
-    (property "Footprint" "TerminalBlock_Phoenix:TerminalBlock_Phoenix_MPT-0,5-2-2.54_1x02_P2.54mm_Horizontal" (id 2) (at 175.26 134.62 0)
+    (property "Footprint" "TerminalBlock_TE-Connectivity:TerminalBlock_TE_282834-2_1x02_P2.54mm_Horizontal" (id 2) (at 175.26 134.62 0)
       (effects (font (size 1.27 1.27)) hide)
     )
@@
       (effects (font (size 1.27 1.27)) (justify left) hide)
     )
-    (pin "1")
-    (pin "2")
-    (pin "5")
     (pin "3")
     (pin "4")
@@
       (effects (font (size 1.27 1.27)) (justify left))
     )
-    (property "Footprint" "TerminalBlock_Phoenix:TerminalBlock_Phoenix_MPT-0,5-2-2.54_1x02_P2.54mm_Horizontal" (id 2) (at 92.71 85.09 0)
+    (property "Footprint" "TerminalBlock_TE-Connectivity:TerminalBlock_TE_282834-2_1x02_P2.54mm_Horizontal" (id 2) (at 92.71 85.09 0)
       (effects (font (size 1.27 1.27)) hide)
     )
@@
       (effects (font (size 1.27 1.27)) (justify left))
     )
-    (property "Footprint" "TerminalBlock_Phoenix:TerminalBlock_Phoenix_MPT-0,5-2-2.54_1x02_P2.54mm_Horizontal" (id 2) (at 175.26 85.09 0)
+    (property "Footprint" "TerminalBlock_TE-Connectivity:TerminalBlock_TE_282834-2_1x02_P2.54mm_Horizontal" (id 2) (at 175.26 85.09 0)
       (effects (font (size 1.27 1.27)) hide)
     )
@@
       (effects (font (size 1.27 1.27)) (justify left))
     )
-    (property "Footprint" "TerminalBlock_Phoenix:TerminalBlock_Phoenix_MPT-0,5-2-2.54_1x02_P2.54mm_Horizontal" (id 2) (at 92.71 135.89 0)
+    (property "Footprint" "TerminalBlock_TE-Connectivity:TerminalBlock_TE_282834-2_1x02_P2.54mm_Horizontal" (id 2) (at 92.71 135.89 0)
       (effects (font (size 1.27 1.27)) hide)
     )
@@
     (pin "2")
     (pin "5")
+  )
+  (symbol (lib_id "KP-PTR_lib:DMC2025UFDB_v2") (at 167.64 74.93 0) (mirror x) (unit 2)
+    (in_bom yes) (on_board yes) (fields_autoplaced)
+    (property "Reference" "Q4" (id 0) (at 172.72 76.835 0)
+      (effects (font (size 1.27 1.27)) (justify left))
+    )
+    (property "Value" "DMC2025UFDB_v2" (id 1) (at 172.72 74.93 0)
+      (effects (font (size 1.27 1.27)) (justify left))
+    )
+    (property "Footprint" "KP-PTR_lib:DMC2025UFDB" (id 2) (at 172.72 73.025 0)
+      (effects (font (size 1.27 1.27)) (justify left) hide)
+    )
+    (property "Datasheet" "http://www.irf.com/product-info/datasheets/data/irf7309ipbf.pdf" (id 3) (at 170.18 74.93 0)
+      (effects (font (size 1.27 1.27)) (justify left) hide)
+    )
     (pin "3")
     (pin "4")
     (pin "6")
   )
-  (symbol (lib_id "KP-PTR_lib:DMC2025UFDB_v2") (at 167.64 74.93 0) (mirror x) (unit 2)
-    (in_bom yes) (on_board yes) (fields_autoplaced)
-    (property "Reference" "Q4" (id 0) (at 172.72 76.835 0)
-      (effects (font (size 1.27 1.27)) (justify left))
-    )
-    (property "Value" "DMC2025UFDB_v2" (id 1) (at 172.72 74.93 0)
-      (effects (font (size 1.27 1.27)) (justify left))
-    )
-    (property "Footprint" "KP-PTR_lib:DMC2025UFDB" (id 2) (at 172.72 73.025 0)
-      (effects (font (size 1.27 1.27)) (justify left) hide)
-    )
-    (property "Datasheet" "http://www.irf.com/product-info/datasheets/data/irf7309ipbf.pdf" (id 3) (at 170.18 74.93 0)
-      (effects (font (size 1.27 1.27)) (justify left) hide)
-    )
-    (pin "1")
-    (pin "2")
-    (pin "5")
-    (pin "3")
-    (pin "4")
-    (pin "6")
-  )
   (symbol (lib_id "Device:R") (at 142.24 99.06 0) (unit 1)
     (in_bom yes) (on_board yes)
@@
     (pin "2")
     (pin "5")
-    (pin "3")
-    (pin "4")
-    (pin "6")
   )
   (symbol (lib_id "power:VCC") (at 170.18 59.69 0) (unit 1)
@@
     (pin "2")
     (pin "5")
-    (pin "3")
-    (pin "4")
-    (pin "6")
   )
   (symbol (lib_id "Device:Polyfuse") (at 170.18 113.03 0) (unit 1)
@@
     (pin "2")
     (pin "5")
-    (pin "3")
-    (pin "4")
-    (pin "6")
   )
   (symbol (lib_id "power:Earth") (at 153.67 87.63 0) (unit 1)
