File: kp-ptr/kp-ptr.kicad_sch (KiCad schematic)
At the start: 29 parts, among them J1 ESP32_PROG_CON, U1 ESP32-S3FN8, Y1 7M40000005-40MHz

Commit message: Grupowanie
Parts:
- renumbered ANT2 to ANT1, C2 to C1, C11 to C10, C12 to C11, C13 to C12, C14 to C13, C15 to C14, C16 to C15, C3 to C2, C4 to C3, C5 to C4, C6 to C5, C7 to C6, C8 to C7, C9 to C8, C10 to C9, L2 to L1, L3 to L2, R2 to R1, R6 to R2, R8 to R3, R14 to R4, R1 to R5, R3 to R6, R4 to R7, R5 to R8

Commit message: PCB update
Parts:
- removed ANT1: PCB_antenna, RF_Antenna:Texas_SWRA117D_2.4GHz_Right, symbol Device:Antenna_Dipole
Changed lines of the file:
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@@
     (pin "4")
-  )
-  (symbol (lib_id "Device:Antenna_Dipole") (at 21.59 48.26 90) (mirror x) (unit 1)
-    (in_bom yes) (on_board yes) (fields_autoplaced)
-    (property "Reference" "ANT1" (id 0) (at 24.13 40.64 90))
-    (property "Value" "PCB_antenna" (id 1) (at 24.13 43.18 90))
-    (property "Footprint" "RF_Antenna:Texas_SWRA117D_2.4GHz_Right" (id 2) (at 21.59 48.26 0)
-      (effects (font (size 1.27 1.27)) hide)
-    )
-    (property "Datasheet" "~" (id 3) (at 21.59 48.26 0)
-      (effects (font (size 1.27 1.27)) hide)
-    )
-    (pin "1")
-    (pin "2")
   )
   (symbol (lib_id "Device:C") (at 228.6 134.62 180) (unit 1)
@@
       (reference "#PWR094") (unit 1) (value "Earth") (footprint "")
     )
-    (path "/f38dad53-0af4-40f6-a173-e0e37aecb5da/c3bf1674-c93f-429b-8563-61b0f5c4ccb1"
-      (reference "#PWR095") (unit 1) (value "VDD") (footprint "")
-    )
     (path "/f38dad53-0af4-40f6-a173-e0e37aecb5da/7bb5e69f-3880-4851-a3bd-776037b6dfcf"
       (reference "#PWR096") (unit 1) (value "Earth") (footprint "")
@@
       (reference "#PWR0132") (unit 1) (value "Earth") (footprint "")
     )
-    (path "/5f9da060-2eb0-4ae6-ad5b-b0da419a62a6/076366eb-2387-4958-8268-f0b75b676a08"
-      (reference "#PWR0133") (unit 1) (value "Earth") (footprint "")
+    (path "/68d9bec4-a8fa-482b-99d8-a42578238d37/9e6cec5d-f256-43fd-a440-00c62c3aeb39"
+      (reference "#PWR0133") (unit 1) (value "+3.3V") (footprint "")
     )
     (path "/5f9da060-2eb0-4ae6-ad5b-b0da419a62a6/5abbc442-e11e-4618-b087-a272d6c9eeca"
@@
       (reference "#PWR0175") (unit 1) (value "Earth") (footprint "")
     )
-    (path "/c5e587d4-4b5f-4f11-98c8-85e16edb877b"
-      (reference "ANT1") (unit 1) (value "PCB_antenna") (footprint "RF_Antenna:Texas_SWRA117D_2.4GHz_Right")
+    (path "/68d9bec4-a8fa-482b-99d8-a42578238d37/862875ce-6e13-42bc-b8a6-de89301ff373"
+      (reference "#PWR0176") (unit 1) (value "+3.3V") (footprint "")
+    )
+    (path "/f38dad53-0af4-40f6-a173-e0e37aecb5da/f5b611b5-22fb-4440-9afb-03e769af8b2d"
+      (reference "#PWR0177") (unit 1) (value "VCC") (footprint "")
     )
     (path "/1d5e7912-4d51-4a4c-b45e-2695b4191d61/2b12b2d4-198b-4c76-b90a-d4d1638b8e72"
       (reference "ANT2") (unit 1) (value "APAE1575R1340ABDD6-T") (footprint "KP-PTR_lib:APAE1575 13x13x4mm GPS Patch Antenna")
     )
-    (path "/5f9da060-2eb0-4ae6-ad5b-b0da419a62a6/911c9e40-8d0a-4a95-a324-f646d3493355"
-      (reference "ANT3") (unit 1) (value "TBD") (footprint "Resistor_SMD:R_0402_1005Metric_Pad0.72x0.64mm_HandSolder")
-    )
     (path "/8ef1d6c2-9afb-467f-94f0-2a571e5715a1"
       (reference "C1") (unit 1) (value "4pF") (footprint "Capacitor_SMD:C_0402_1005Metric")
@@
       (reference "C26") (unit 1) (value "1nF") (footprint "Capacitor_SMD:C_0402_1005Metric")
     )
-    (path "/1d5e7912-4d51-4a4c-b45e-2695b4191d61/5e346ddf-4399-45f3-970a-1479f18e976f"
-      (reference "C27") (unit 1) (value "DNP") (footprint "Capacitor_SMD:C_0402_1005Metric")
-    )
     (path "/1d5e7912-4d51-4a4c-b45e-2695b4191d61/f96866fb-2dc5-44d0-95c9-2f03b948fe38"
       (reference "C28") (unit 1) (value "10uF") (footprint "Capacitor_SMD:C_0402_1005Metric")
@@
     )
     (path "/f38dad53-0af4-40f6-a173-e0e37aecb5da/ceb2713e-b9d7-42d2-af1c-a38a6fc43b0d"
-      (reference "C34") (unit 1) (value "TBD") (footprint "Capacitor_SMD:C_0402_1005Metric")
+      (reference "C34") (unit 1) (value "TBD") (footprint "Capacitor_SMD:CP_Elec_10x10")
     )
     (path "/f38dad53-0af4-40f6-a173-e0e37aecb5da/b3fe89b5-5813-4c35-a55a-fe0f40d2e320"
@@
     )
     (path "/1d5e7912-4d51-4a4c-b45e-2695b4191d61/ffd6a983-4822-4f37-978e-177b7febe08c"
-      (reference "D2") (unit 1) (value "TBD") (footprint "Diode_SMD:D_SOD-123")
+      (reference "D2") (unit 1) (value "TBD") (footprint "Diode_SMD:D_0402_1005Metric")
     )
     (path "/f38dad53-0af4-40f6-a173-e0e37aecb5da/55b5f7c1-9e27-4de8-8da9-4ddd7c634c2f"
@@
     )
     (path "/5f9da060-2eb0-4ae6-ad5b-b0da419a62a6/94e53db9-ffab-45c9-951c-83988bceb04a"
-      (reference "D9") (unit 1) (value "TBD") (footprint "Diode_SMD:D_SOD-123")
+      (reference "D9") (unit 1) (value "TBD") (footprint "Diode_SMD:D_0402_1005Metric")
     )
     (path "/68d9bec4-a8fa-482b-99d8-a42578238d37/7419015c-d6f5-473a-81b5-0c1550cbc74a"
@@
     )
     (path "/5f9da060-2eb0-4ae6-ad5b-b0da419a62a6/ed569010-9483-41f9-9593-9fb3bab33022"
-      (reference "J4") (unit 1) (value "USB_C_Receptacle_USB2.0") (footprint "Connector_USB:USB_C_Receptacle_GCT_USB4085")
+      (reference "J4") (unit 1) (value "USB_C_Receptacle_USB2.0") (footprint "KP-PTR_lib:USB_C_213716")
     )
     (path "/5f9da060-2eb0-4ae6-ad5b-b0da419a62a6/51441429-c522-44d6-becc-0386208970a8"
-      (reference "J5") (unit 1) (value "u.fl") (footprint "Connector_Coaxial:U.FL_Hirose_U.FL-R-SMT-1_Vertical")
+      (reference "J5") (unit 1) (value "u.fl") (footprint "Connector_Coaxial:SMA_Amphenol_132289_EdgeMount")
     )
     (path "/68d9bec4-a8fa-482b-99d8-a42578238d37/c390b41f-5a60-4177-8299-f081c7daef82"
@@
     )
     (path "/f38dad53-0af4-40f6-a173-e0e37aecb5da/51187671-afc4-4b52-80d4-111c6700a75a"
-      (reference "R21") (unit 1) (value "DNP") (footprint "Resistor_SMD:R_0402_1005Metric")
+      (reference "R21") (unit 1) (value "DNP") (footprint "Resistor_SMD:R_1206_3216Metric")
     )
     (path "/f38dad53-0af4-40f6-a173-e0e37aecb5da/0bae5ae7-8423-4396-8155-8b7564351343"
@@
       (reference "R26") (unit 1) (value "100k") (footprint "Resistor_SMD:R_0402_1005Metric")
     )
-    (path "/5f9da060-2eb0-4ae6-ad5b-b0da419a62a6/db0c09fb-ffc7-40ad-a12a-7d061e659129"
-      (reference "R27") (unit 1) (value "100k") (footprint "Resistor_SMD:R_0402_1005Metric")
+    (path "/68d9bec4-a8fa-482b-99d8-a42578238d37/2550be30-43c7-4aff-b035-90fec992dc6d"
+      (reference "R27") (unit 1) (value "10k") (footprint "Resistor_SMD:R_0402_1005Metric")
     )
     (path "/5f9da060-2eb0-4ae6-ad5b-b0da419a62a6/eebca155-80f9-46f5-916f-1a12a740217b"
@@
       (reference "R31") (unit 1) (value "10k") (footprint "Resistor_SMD:R_0402_1005Metric")
     )
-    (path "/5f9da060-2eb0-4ae6-ad5b-b0da419a62a6/96060ebb-a1ce-4017-966f-a8a530fafaf5"
-      (reference "R32") (unit 1) (value "DNP") (footprint "Resistor_SMD:R_0402_1005Metric")
-    )
-    (path "/5f9da060-2eb0-4ae6-ad5b-b0da419a62a6/ac606df2-b12e-4b6f-b98c-485616a18436"
-      (reference "R33") (unit 1) (value "0R") (footprint "Resistor_SMD:R_0402_1005Metric")
+    (path "/68d9bec4-a8fa-482b-99d8-a42578238d37/4ec3a6b7-bbcd-44f9-bc96-f5fd8d503e96"
+      (reference "R32") (unit 1) (value "10k") (footprint "Resistor_SMD:R_0402_1005Metric")
     )
     (path "/68d9bec4-a8fa-482b-99d8-a42578238d37/731faaa8-00a4-4456-82f6-d47cf24c2880"

Commit message: SCH&PCB update
Parts:
- added AE1: Antenna_Chip, KP-PTR_lib:AMCA31-2R450G-S1F-T3, symbol Device:Antenna_Chip
Connections:
- net GPIO1 is gone; now on net GPS_IN: U1.6 (GPIO1/ADC1_CH0)
- net GPIO10 is gone; now on net IGN2_EN: U1.15 (GPIO10/ADC1_CH9)
- net GPIO11 is gone; now on net IGN1_EN: U1.16 (GPIO11/ADC2_CH0)
- net GPIO12 is gone; now on net IGN4_EN: U1.17 (GPIO12/ADC2_CH1)
- net GPIO13 is gone; now on net UART1_OUT: U1.18 (GPIO13/ADC2_CH2)
- net GPIO14 is gone; now on net UART1_IN: U1.19 (GPIO14/ADC2_CH3)
- net GPIO15 is gone; now on net I2C_SDA: U1.21 (GPIO15/ADC2_CH4/XTAL_32K_P)
- net GPIO16 is gone; now on net I2C_SCL: U1.22 (GPIO16/ADC2_CH5/XTAL_32K_N)
- net GPIO17 is gone; now on net SERVO_1: U1.23 (GPIO17/ADC2_CH6/DAC_2)
- net GPIO18 is gone; now on net SERVO_2: U1.24 (GPIO18/ADC2_CH7/DAC_1)
- net GPIO2 is gone; now on net GPS_OUT: U1.7 (GPIO2/ADC1_CH1)
- net GPIO21 is gone; now on net SERVO_3: U1.27 (GPIO21)
- net GPIO26 is gone; now on net SERVO_4: U1.28 (SPI_CS1/GPIO26)
- net GPIO33 is gone; now on net SPI_CS_FLASH: U1.38 (GPIO33)
- net GPIO34 is gone; now on net SPI_CS_MAG: U1.39 (GPIO34)
- net GPIO35 is gone; now on net SPI_CS_LSM: U1.40 (GPIO35)
- net GPIO36 is gone; now on net SPI_CS_LIS: U1.41 (GPIO36)
- net GPIO37 is gone; now on net RF_BUSY: U1.42 (GPIO37)
- net GPIO38 is gone; now on net SPI_MISO: U1.43 (GPIO38)
- net GPIO39 is gone; now on net SPI_MOSI: U1.44 (MTCK/JTAG/GPIO39)
- net GPIO4 is gone; now on net IGN4_DET: U1.9 (GPIO4/ADC1_CH3)
- net GPIO40 is gone; now on net SPI_CLK: U1.45 (MTDO/JTAG/GPIO40)
- net GPIO41 is gone; now on net SPI_CS_MS5607: U1.47 (MTDI/JTAG/GPIO41)
- net GPIO42 is gone; now on net SPI_CS_LORA: U1.48 (MTMS/JTAG/GPIO42)
- net GPIO47 is gone; now on net LED1: U1.37 (SPICLK_P/GPIO47)
- net GPIO48 is gone; now on net SERVO_EN: U1.36 (SPICLK_N/GPIO48)
- net GPIO5 is gone; now on net IGN1_DET: U1.10 (GPIO5/ADC1_CH4)
- net GPIO6 is gone; now on net IGN2_DET: U1.11 (GPIO6/ADC1_CH5)
- net GPIO7 is gone; now on net IGN3_DET: U1.12 (GPIO7/ADC1_CH6)
- net GPIO8 is gone; now on net VBAT_MEAS: U1.13 (GPIO8/ADC1_CH7)
- net GPIO9 is gone; now on net IGN3_EN: U1.14 (GPIO9/ADC1_CH8)
- net at C1.1, L1.1: now also AE1.2 (PCB_Trace)

Commit message: Footprints and PCB update
Connections:
- net at C1.1, L1.1: now also AE1.1 (FEED); no longer AE1.2 (PCB_Trace)
Other:
- moved on the sheet: AE1
Changed lines of the file:
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@@
     (pin "2")
   )
-  (symbol (lib_id "Device:Antenna_Chip") (at 24.13 45.72 0) (unit 1)
+  (symbol (lib_id "Device:Antenna_Chip") (at 24.13 45.72 0) (mirror y) (unit 1)
     (in_bom yes) (on_board yes) (fields_autoplaced)
-    (property "Reference" "AE1" (id 0) (at 29.21 41.9099 0)
-      (effects (font (size 1.27 1.27)) (justify left))
+    (property "Reference" "AE1" (id 0) (at 27.94 41.9099 0)
+      (effects (font (size 1.27 1.27)) (justify right))
     )
-    (property "Value" "Antenna_Chip" (id 1) (at 29.21 44.4499 0)
-      (effects (font (size 1.27 1.27)) (justify left))
+    (property "Value" "Antenna_Chip" (id 1) (at 27.94 44.4499 0)
+      (effects (font (size 1.27 1.27)) (justify right))
     )
-    (property "Footprint" "KP-PTR_lib:AMCA31-2R450G-S1F-T3" (id 2) (at 21.59 41.275 0)
+    (property "Footprint" "KP-PTR_lib:AMCA31-2R450G-S1F-T3" (id 2) (at 26.67 41.275 0)
       (effects (font (size 1.27 1.27)) hide)
     )
-    (property "Datasheet" "~" (id 3) (at 21.59 41.275 0)
+    (property "Datasheet" "~" (id 3) (at 26.67 41.275 0)
       (effects (font (size 1.27 1.27)) hide)
     )

Commit message: Update from v0.1 to v1.0
Parts:
- C3: footprint Capacitor_SMD:C_0402_1005Metric -> Capacitor_SMD:C_0603_1608Metric
- R5: value 1k -> 10k
Changed lines of the file:
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@@
     (in_bom yes) (on_board yes)
     (property "Reference" "R5" (id 0) (at 63.5 170.18 90))
-    (property "Value" "1k" (id 1) (at 58.42 170.18 90))
+    (property "Value" "10k" (id 1) (at 58.42 170.18 90))
     (property "Footprint" "Resistor_SMD:R_0402_1005Metric" (id 2) (at 62.738 171.45 90)
       (effects (font (size 1.27 1.27)) hide)
@@
       (effects (font (size 1.27 1.27)) (justify left))
     )
-    (property "Footprint" "Capacitor_SMD:C_0402_1005Metric" (id 2) (at 58.1152 133.35 0)
+    (property "Footprint" "Capacitor_SMD:C_0603_1608Metric" (id 2) (at 58.1152 133.35 0)
       (effects (font (size 1.27 1.27)) hide)
     )
@@
     )
     (path "/4f1274ca-1a6c-4d3f-a67e-a17628c6ce80"
-      (reference "C3") (unit 1) (value "10u") (footprint "Capacitor_SMD:C_0402_1005Metric")
+      (reference "C3") (unit 1) (value "10u") (footprint "Capacitor_SMD:C_0603_1608Metric")
     )
     (path "/bc35207d-1b8c-4995-a83a-f31026da2155"
@@
     )
     (path "/1d5e7912-4d51-4a4c-b45e-2695b4191d61/e96c3e2a-2126-4340-898b-967da0484374"
-      (reference "C16") (unit 1) (value "10uF") (footprint "Capacitor_SMD:C_0402_1005Metric")
+      (reference "C16") (unit 1) (value "10uF") (footprint "Capacitor_SMD:C_0603_1608Metric")
     )
     (path "/1d5e7912-4d51-4a4c-b45e-2695b4191d61/3692f320-6cad-4720-a461-3a4196de5452"
@@
     )
     (path "/1d5e7912-4d51-4a4c-b45e-2695b4191d61/14236b38-4ab2-40f1-8dab-acd37ddaabd5"
-      (reference "C20") (unit 1) (value "10uF") (footprint "Capacitor_SMD:C_0402_1005Metric")
+      (reference "C20") (unit 1) (value "10uF") (footprint "Capacitor_SMD:C_0603_1608Metric")
     )
     (path "/1d5e7912-4d51-4a4c-b45e-2695b4191d61/f1b6778f-fb59-42c5-ab69-9aeffa407186"
@@
     )
     (path "/1d5e7912-4d51-4a4c-b45e-2695b4191d61/26845ef0-0144-4941-baba-e09c06b1135e"
-      (reference "C23") (unit 1) (value "4.7uF") (footprint "Capacitor_SMD:C_0402_1005Metric")
+      (reference "C23") (unit 1) (value "10uF") (footprint "Capacitor_SMD:C_0603_1608Metric")
     )
     (path "/1d5e7912-4d51-4a4c-b45e-2695b4191d61/cf4d831e-5df7-407d-8087-3427973fbcc4"
-      (reference "C24") (unit 1) (value "4.7uF") (footprint "Capacitor_SMD:C_0402_1005Metric")
+      (reference "C24") (unit 1) (value "10uF") (footprint "Capacitor_SMD:C_0603_1608Metric")
     )
     (path "/1d5e7912-4d51-4a4c-b45e-2695b4191d61/c2375d21-e2a2-4412-ae36-ccb229323597"
-      (reference "C25") (unit 1) (value "56pF") (footprint "Capacitor_SMD:C_0402_1005Metric")
+      (reference "C25") (unit 1) (value "DNP") (footprint "Capacitor_SMD:C_0402_1005Metric")
     )
     (path "/1d5e7912-4d51-4a4c-b45e-2695b4191d61/cb8b5a4d-f53c-4fdd-bbba-ccb732fe5d61"
@@
     )
     (path "/1d5e7912-4d51-4a4c-b45e-2695b4191d61/f96866fb-2dc5-44d0-95c9-2f03b948fe38"
-      (reference "C28") (unit 1) (value "10uF") (footprint "Capacitor_SMD:C_0402_1005Metric")
+      (reference "C28") (unit 1) (value "10uF") (footprint "Capacitor_SMD:C_0603_1608Metric")
     )
     (path "/1d5e7912-4d51-4a4c-b45e-2695b4191d61/6dcb165b-9b58-46a2-ba9c-c210aaff5476"
@@
     )
     (path "/1d5e7912-4d51-4a4c-b45e-2695b4191d61/b8207dfe-6211-4bc0-9abf-df9bab15cfb2"
-      (reference "C30") (unit 1) (value "DNP") (footprint "Capacitor_SMD:C_0402_1005Metric")
+      (reference "C30") (unit 1) (value "56pF") (footprint "Capacitor_SMD:C_0402_1005Metric")
     )
     (path "/1d5e7912-4d51-4a4c-b45e-2695b4191d61/a9c75ea3-896c-4808-8937-ae3cbc60880e"
@@
     )
     (path "/f38dad53-0af4-40f6-a173-e0e37aecb5da/b3fe89b5-5813-4c35-a55a-fe0f40d2e320"
-      (reference "C35") (unit 1) (value "10u") (footprint "Capacitor_SMD:C_0402_1005Metric")
+      (reference "C35") (unit 1) (value "10uF 6V3") (footprint "Capacitor_SMD:C_0603_1608Metric")
     )
     (path "/f38dad53-0af4-40f6-a173-e0e37aecb5da/4c0f4562-338e-4c3f-8e5e-d190dafff1ba"
-      (reference "C36") (unit 1) (value "10u") (footprint "Capacitor_SMD:C_0402_1005Metric")
+      (reference "C36") (unit 1) (value "10uF 6V3") (footprint "Capacitor_SMD:C_0603_1608Metric")
     )
     (path "/f38dad53-0af4-40f6-a173-e0e37aecb5da/8ff4940c-12aa-47f7-a118-efe963b3599f"
-      (reference "C37") (unit 1) (value "1uF") (footprint "Capacitor_SMD:C_0402_1005Metric")
+      (reference "C37") (unit 1) (value "100n") (footprint "Capacitor_SMD:C_0402_1005Metric")
     )
     (path "/f38dad53-0af4-40f6-a173-e0e37aecb5da/c5a597f4-0866-4388-bce4-7fa670e3ab69"
-      (reference "C38") (unit 1) (value "1uF") (footprint "Capacitor_SMD:C_0402_1005Metric")
+      (reference "C38") (unit 1) (value "100n 50V") (footprint "Capacitor_SMD:C_0402_1005Metric")
     )
     (path "/5f9da060-2eb0-4ae6-ad5b-b0da419a62a6/f61a552a-1c8d-4e4a-a497-ddf53496bf6e"
@@
     )
     (path "/5f9da060-2eb0-4ae6-ad5b-b0da419a62a6/6c16042f-ade1-413e-a421-4ab855737deb"
-      (reference "C43") (unit 1) (value "4u7") (footprint "Capacitor_SMD:C_0402_1005Metric")
+      (reference "C43") (unit 1) (value "10uF") (footprint "Capacitor_SMD:C_0603_1608Metric")
     )
     (path "/68d9bec4-a8fa-482b-99d8-a42578238d37/a507659a-1b9c-4e3d-98a6-2c6f6ba0f0bf"
@@
     )
     (path "/6b0b54eb-96fb-4a56-9d20-0b579f8bbc83/a4f64921-f3d5-4c46-878a-337a6c787dd8"
-      (reference "C47") (unit 1) (value "TBD") (footprint "Capacitor_SMD:C_0402_1005Metric")
+      (reference "C47") (unit 1) (value "1uF") (footprint "Capacitor_SMD:C_0402_1005Metric")
     )
     (path "/6b0b54eb-96fb-4a56-9d20-0b579f8bbc83/be63f366-5326-4f66-bf46-d15339c7c67e"
-      (reference "C48") (unit 1) (value "TBD") (footprint "Capacitor_SMD:C_0402_1005Metric")
+      (reference "C48") (unit 1) (value "1uF") (footprint "Capacitor_SMD:C_0402_1005Metric")
     )
     (path "/6b0b54eb-96fb-4a56-9d20-0b579f8bbc83/86cd46fa-0d03-4ab7-bf27-02e71711b288"
-      (reference "C49") (unit 1) (value "TBD") (footprint "Capacitor_SMD:C_0402_1005Metric")
+      (reference "C49") (unit 1) (value "1uF") (footprint "Capacitor_SMD:C_0402_1005Metric")
     )
     (path "/6b0b54eb-96fb-4a56-9d20-0b579f8bbc83/3ad9e242-3293-49dd-9a86-c609234e3bcf"
-      (reference "C50") (unit 1) (value "TBD") (footprint "Capacitor_SMD:C_0402_1005Metric")
+      (reference "C50") (unit 1) (value "1uF") (footprint "Capacitor_SMD:C_0402_1005Metric")
     )
     (path "/1d5e7912-4d51-4a4c-b45e-2695b4191d61/c0e01ba5-ed56-4572-a513-e7708605b1ff"
@@
     )
     (path "/f38dad53-0af4-40f6-a173-e0e37aecb5da/413bd791-2789-4ff7-be50-3aae609090d4"
-      (reference "F1") (unit 1) (value "500mA") (footprint "Fuse:Fuse_0805_2012Metric")
+      (reference "F1") (unit 1) (value "500mA") (footprint "Fuse:Fuse_1210_3225Metric")
     )
     (path "/6b0b54eb-96fb-4a56-9d20-0b579f8bbc83/b976339d-e23f-413f-9e9d-e93e2b444e20"
-      (reference "F2") (unit 1) (value "500mA") (footprint "Fuse:Fuse_0805_2012Metric")
+      (reference "F2") (unit 1) (value "500mA") (footprint "Fuse:Fuse_1210_3225Metric")
     )
     (path "/6b0b54eb-96fb-4a56-9d20-0b579f8bbc83/ceef1b14-dada-4cd1-baac-ef03c2509802"
-      (reference "F3") (unit 1) (value "500mA") (footprint "Fuse:Fuse_0805_2012Metric")
+      (reference "F3") (unit 1) (value "500mA") (footprint "Fuse:Fuse_1210_3225Metric")
     )
     (path "/6b0b54eb-96fb-4a56-9d20-0b579f8bbc83/7170860f-7531-424c-b87d-f03c82085b5e"
-      (reference "F4") (unit 1) (value "500mA") (footprint "Fuse:Fuse_0805_2012Metric")
+      (reference "F4") (unit 1) (value "500mA") (footprint "Fuse:Fuse_1210_3225Metric")
     )
     (path "/6b0b54eb-96fb-4a56-9d20-0b579f8bbc83/d5754530-1e98-486a-8e5a-977de4a011bd"
-      (reference "F5") (unit 1) (value "500mA") (footprint "Fuse:Fuse_0805_2012Metric")
+      (reference "F5") (unit 1) (value "500mA") (footprint "Fuse:Fuse_1210_3225Metric")
     )
     (path "/1d5e7912-4d51-4a4c-b45e-2695b4191d61/267f3f5c-5986-42a8-90e0-9867572b9498"
@@
     )
     (path "/2c7c4624-5556-4f0a-9902-0e418133e1f8"
-      (reference "R5") (unit 1) (value "1k") (footprint "Resistor_SMD:R_0402_1005Metric")
+      (reference "R5") (unit 1) (value "10k") (footprint "Resistor_SMD:R_0402_1005Metric")
     )
     (path "/754b6893-1907-4e64-812a-fb1b4644d93e"
@@
     )
     (path "/f38dad53-0af4-40f6-a173-e0e37aecb5da/ebfd6638-c4a6-4b93-8160-3b3910e87fd4"
-      (reference "R19") (unit 1) (value "100k") (footprint "Resistor_SMD:R_0402_1005Metric")
+      (reference "R19") (unit 1) (value "100k 1%") (footprint "Resistor_SMD:R_0402_1005Metric")
     )
     (path "/f38dad53-0af4-40f6-a173-e0e37aecb5da/501992b5-b8b1-4742-aa03-cb1dabac6355"
-      (reference "R20") (unit 1) (value "10k") (footprint "Resistor_SMD:R_0402_1005Metric")
+      (reference "R20") (unit 1) (value "10k 1%") (footprint "Resistor_SMD:R_0402_1005Metric")
     )
     (path "/f38dad53-0af4-40f6-a173-e0e37aecb5da/51187671-afc4-4b52-80d4-111c6700a75a"
@@
     )
     (path "/f38dad53-0af4-40f6-a173-e0e37aecb5da/02ab2548-d360-4d53-ba49-ccf0853e38ce"
-      (reference "R23") (unit 1) (value "20k") (footprint "Resistor_SMD:R_0402_1005Metric")
+      (reference "R23") (unit 1) (value "22k") (footprint "Resistor_SMD:R_0402_1005Metric")
     )
     (path "/f38dad53-0af4-40f6-a173-e0e37aecb5da/3480cc69-0d8f-4c1a-a184-a2c19d600374"
@@
     )
     (path "/5f9da060-2eb0-4ae6-ad5b-b0da419a62a6/42e6c123-deaa-49d0-9568-19cbdde78d54"
-      (reference "R26") (unit 1) (value "100k") (footprint "Resistor_SMD:R_0402_1005Metric")
+      (reference "R26") (unit 1) (value "10k") (footprint "Resistor_SMD:R_0402_1005Metric")
     )
     (path "/68d9bec4-a8fa-482b-99d8-a42578238d37/2550be30-43c7-4aff-b035-90fec992dc6d"
