File: kp-ptr/sensors.kicad_sch (KiCad schematic)
At the start: 38 parts, among them U3 MS560702BA03-50, U4 MMC5983MA, U5 H3LIS331, U6 L76-L, U7 LSM6DSO32, U9 NJG1156PCD

Commit message: Kilka zmian.
-dodany tranzystor P/N mosfet do biblioteki i zapalników
-dodany komentarz o impedancji ścieżek RF
Parts:
- ANT?: footprint (none) -> KP-PTR_lib:APAE1575 13x13x4mm GPS Patch Antenna
Other:
- note added: "50 Ohm"
Changed lines of the file:
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@@
+    (effects (font (size 1.27 1.27)) (justify left bottom))
+  )
+  (text "50 Ohm" (at 190.5 130.81 0)
     (effects (font (size 1.27 1.27)) (justify left bottom))
   )
@@
     (effects (font (size 1.27 1.27)) (justify left bottom))
   )
+  (text "50 Ohm" (at 261.62 135.89 0)
+    (effects (font (size 1.27 1.27)) (justify left bottom))
+  )
   (text "GPS" (at 114.3 101.6 0)
+    (effects (font (size 1.27 1.27)) (justify left bottom))
+  )
+  (text "50 Ohm" (at 207.01 127 0)
+    (effects (font (size 1.27 1.27)) (justify left bottom))
+  )
+  (text "50 Ohm" (at 224.79 118.11 0)
     (effects (font (size 1.27 1.27)) (justify left bottom))
   )
@@
       (effects (font (size 1.27 1.27)) (justify left))
     )
-    (property "Footprint" "" (id 2) (at 270.51 130.81 0)
-      (effects (font (size 1.27 1.27)) hide)
-    )
+    (property "Footprint" "KP-PTR_lib:APAE1575 13x13x4mm GPS Patch Antenna" (id 2) (at 270.51 130.81 0)
+      (effects (font (size 1.27 1.27)) hide)
+    )

Commit message: Szlifowanie schematu
Connections:
- net U0RXD renamed GPS_OUT
- net U0TXD renamed GPS_IN
Changed lines of the file:
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@@
     )
   )
-  (global_label "U0TXD" (shape input) (at 120.65 135.89 180) (fields_autoplaced)
+  (global_label "GPS_IN" (shape input) (at 120.65 135.89 180) (fields_autoplaced)
     (effects (font (size 1.27 1.27)) (justify right))
-    (property "Intersheet References" "${INTERSHEET_REFS}" (id 0) (at 112.2498 135.8106 0)
+    (property "Intersheet References" "${INTERSHEET_REFS}" (id 0) (at 111.5845 135.8106 0)
       (effects (font (size 1.27 1.27)) (justify right) hide)
     )
@@
     )
   )
-  (global_label "U0RXD" (shape input) (at 121.92 143.51 180) (fields_autoplaced)
+  (global_label "GPS_OUT" (shape input) (at 121.92 143.51 180) (fields_autoplaced)
     (effects (font (size 1.27 1.27)) (justify right))
-    (property "Intersheet References" "${INTERSHEET_REFS}" (id 0) (at 113.2174 143.4306 0)
+    (property "Intersheet References" "${INTERSHEET_REFS}" (id 0) (at 111.1612 143.4306 0)
       (effects (font (size 1.27 1.27)) (justify right) hide)
     )

Commit message: Update po spotkaniu
Parts:
- removed F?: 200mA, symbol Device:Polyfuse
- added FB1: 200mA, Resistor_SMD:R_0402_1005Metric, symbol Device:FerriteBead
- C1, C18, C19, C34, C43: renamed from C?; footprint Capacitor_SMD:C_0402_1005Metric_Pad0.74x0.62mm_HandSolder -> Capacitor_SMD:C_0402_1005Metric
- C17, C20, C21, C22, C23, C24, C25, C26, C27, C28, C29, C30: footprint Capacitor_SMD:C_0402_1005Metric_Pad0.74x0.62mm_HandSolder -> Capacitor_SMD:C_0402_1005Metric
- D1: renamed from D?; footprint LED_SMD:LED_0603_1608Metric_Pad1.05x0.95mm_HandSolder -> LED_SMD:LED_0603_1608Metric
- D6: renamed from D?; footprint (none) -> Diode_SMD:D_SOD-123
- L5: footprint Inductor_SMD:L_0402_1005Metric_Pad0.77x0.64mm_HandSolder -> Inductor_SMD:L_0402_1005Metric
- R15, R16, R21, R22: renamed from R?; footprint Resistor_SMD:R_0402_1005Metric_Pad0.72x0.64mm_HandSolder -> Resistor_SMD:R_0402_1005Metric
- R17, R18, R19, R20, R7, R9: footprint Resistor_SMD:R_0402_1005Metric_Pad0.72x0.64mm_HandSolder -> Resistor_SMD:R_0402_1005Metric
- gave numbers to parts that had none: 1
Connections:
- net +3V3: now also FB1.1; no longer C18.2, C26.1, C27.1, U9.3 (VDD)
- net +3.3VADC: now reaches U6.6 (V_BCKP), U6.8 (VCC)
- net +3.3VADC: now also C18.2, C26.1, C27.1, U9.3 (VDD), FB1.2
Other:
- moved on the sheet: ANT3, C1, C18, C19, C34, C43, D6, L5, R21, R22, U9

Commit message: Grupowanie
Parts:
- renumbered ANT3 to ANT2, C20 to C16, C21 to C17, C22 to C18, C17 to C19, C23 to C20, C24 to C21, C25 to C22, C26 to C23, C27 to C24, C1 to C25, C18 to C26, C19 to C27, C34 to C30, C30 to C31, C43 to C32, D6 to D2, L5 to L3, R17 to R10, R18 to R11, R15 to R12, R19 to R13, R16 to R14, R20 to R15, R21 to R16, R22 to R17, R9 to R18, R7 to R9, U3 to U2, U4 to U3, U5 to U4, U6 to U5, U9 to U6
Connections:
- net Earth: now also U6.6 (GND)

Commit message: PCB update
Parts:
- removed C27: DNP, Capacitor_SMD:C_0402_1005Metric, symbol Device:C
- D2: footprint Diode_SMD:D_SOD-123 -> Diode_SMD:D_0402_1005Metric
Connections:
- net at ANT2.1 (A), C32.1, D2.2 (A2): now also C30.1
- net at C32.2, U6.5 (Pre/IN): no longer C30.1
- net at C25.2, U5.11 (RF_IN): now also C30.2
Other:
- moved on the sheet: C30
Changed lines of the file:
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@@
   (junction (at 38.1 134.62) (diameter 0) (color 0 0 0 0)
   )
+  (junction (at 198.12 130.81) (diameter 0) (color 0 0 0 0)
+  )
   (junction (at 130.81 59.69) (diameter 0) (color 0 0 0 0)
   )
-  (junction (at 248.285 140.97) (diameter 0) (color 0 0 0 0)
-  )
   (junction (at 203.835 137.16) (diameter 0) (color 0 0 0 0)
   )
@@
   (junction (at 130.81 57.15) (diameter 0) (color 0 0 0 0)
   )
+  (junction (at 260.985 140.97) (diameter 0) (color 0 0 0 0)
+  )
   (junction (at 130.81 39.37) (diameter 0) (color 0 0 0 0)
   )
@@
   )
   (junction (at 254 46.99) (diameter 0) (color 0 0 0 0)
-  )
-  (junction (at 217.805 130.81) (diameter 0) (color 0 0 0 0)
   )
   (junction (at 222.25 39.37) (diameter 0) (color 0 0 0 0)
@@
     (stroke (width 0) (type default) (color 0 0 0 0))
   )
+  (wire (pts (xy 253.365 130.81) (xy 222.25 130.81))
+    (stroke (width 0) (type default) (color 0 0 0 0))
+  )
   (wire (pts (xy 36.83 147.32) (xy 36.83 149.86))
     (stroke (width 0) (type default) (color 0 0 0 0))
@@
     (stroke (width 0) (type default) (color 0 0 0 0))
   )
+  (wire (pts (xy 260.985 130.81) (xy 260.985 140.97))
+    (stroke (width 0) (type default) (color 0 0 0 0))
+  )
   (wire (pts (xy 130.81 44.45) (xy 135.89 44.45))
     (stroke (width 0) (type default) (color 0 0 0 0))
@@
     (stroke (width 0) (type default) (color 0 0 0 0))
   )
+  (wire (pts (xy 198.12 120.65) (xy 198.12 130.81))
+    (stroke (width 0) (type default) (color 0 0 0 0))
+  )
   (wire (pts (xy 254 46.99) (xy 257.81 46.99))
     (stroke (width 0) (type default) (color 0 0 0 0))
@@
     (stroke (width 0) (type default) (color 0 0 0 0))
   )
-  (wire (pts (xy 248.285 140.97) (xy 253.365 140.97))
+  (wire (pts (xy 243.205 140.97) (xy 253.365 140.97))
     (stroke (width 0) (type default) (color 0 0 0 0))
   )
@@
     (stroke (width 0) (type default) (color 0 0 0 0))
   )
-  (wire (pts (xy 243.205 140.97) (xy 248.285 140.97))
-    (stroke (width 0) (type default) (color 0 0 0 0))
-  )
   (wire (pts (xy 35.56 142.24) (xy 40.64 142.24))
     (stroke (width 0) (type default) (color 0 0 0 0))
@@
     (stroke (width 0) (type default) (color 0 0 0 0))
   )
-  (wire (pts (xy 217.805 123.19) (xy 248.285 123.19))
-    (stroke (width 0) (type default) (color 0 0 0 0))
-  )
   (wire (pts (xy 120.65 135.89) (xy 125.73 135.89))
     (stroke (width 0) (type default) (color 0 0 0 0))
@@
     (stroke (width 0) (type default) (color 0 0 0 0))
   )
+  (wire (pts (xy 198.12 130.81) (xy 198.755 130.81))
+    (stroke (width 0) (type default) (color 0 0 0 0))
+  )
   (wire (pts (xy 251.46 52.07) (xy 252.73 52.07))
     (stroke (width 0) (type default) (color 0 0 0 0))
@@
     (stroke (width 0) (type default) (color 0 0 0 0))
   )
+  (wire (pts (xy 198.12 120.65) (xy 222.25 120.65))
+    (stroke (width 0) (type default) (color 0 0 0 0))
+  )
   (wire (pts (xy 222.25 41.91) (xy 222.25 39.37))
     (stroke (width 0) (type default) (color 0 0 0 0))
@@
     (stroke (width 0) (type default) (color 0 0 0 0))
   )
-  (wire (pts (xy 248.285 130.81) (xy 248.285 140.97))
-    (stroke (width 0) (type default) (color 0 0 0 0))
-  )
   (wire (pts (xy 125.095 114.3) (xy 128.905 114.3))
     (stroke (width 0) (type default) (color 0 0 0 0))
@@
     (stroke (width 0) (type default) (color 0 0 0 0))
   )
-  (wire (pts (xy 191.77 130.81) (xy 198.755 130.81))
+  (wire (pts (xy 191.77 130.81) (xy 198.12 130.81))
     (stroke (width 0) (type default) (color 0 0 0 0))
   )
@@
   )
   (wire (pts (xy 146.05 143.51) (xy 151.13 143.51))
+    (stroke (width 0) (type default) (color 0 0 0 0))
+  )
+  (wire (pts (xy 222.25 130.81) (xy 222.25 120.65))
     (stroke (width 0) (type default) (color 0 0 0 0))
   )
@@
     )
     (pin "1")
-  )
-  (symbol (lib_id "Device:C") (at 217.805 127 180) (unit 1)
-    (in_bom yes) (on_board yes)
-    (property "Reference" "C27" (id 0) (at 213.995 127 90))
-    (property "Value" "DNP" (id 1) (at 221.615 127 90))
-    (property "Footprint" "Capacitor_SMD:C_0402_1005Metric" (id 2) (at 216.8398 123.19 0)
-      (effects (font (size 1.27 1.27)) hide)
-    )
-    (property "Datasheet" "~" (id 3) (at 217.805 127 0)
-      (effects (font (size 1.27 1.27)) hide)
-    )
-    (pin "1")
-    (pin "2")
   )
   (symbol (lib_id "power:Earth") (at 211.455 153.67 0) (unit 1)
@@
     (pin "1")
   )
-  (symbol (lib_id "Device:C") (at 248.285 127 180) (unit 1)
-    (in_bom yes) (on_board yes)
-    (property "Reference" "C30" (id 0) (at 244.475 127 90))
-    (property "Value" "DNP" (id 1) (at 252.095 127 90))
-    (property "Footprint" "Capacitor_SMD:C_0402_1005Metric" (id 2) (at 247.3198 123.19 0)
-      (effects (font (size 1.27 1.27)) hide)
-    )
-    (property "Datasheet" "~" (id 3) (at 248.285 127 0)
+  (symbol (lib_id "Device:C") (at 257.175 130.81 270) (unit 1)
+    (in_bom yes) (on_board yes)
+    (property "Reference" "C30" (id 0) (at 257.175 134.62 90))
+    (property "Value" "DNP" (id 1) (at 257.175 127 90))
+    (property "Footprint" "Capacitor_SMD:C_0402_1005Metric" (id 2) (at 253.365 131.7752 0)
+      (effects (font (size 1.27 1.27)) hide)
+    )
+    (property "Datasheet" "~" (id 3) (at 257.175 130.81 0)
       (effects (font (size 1.27 1.27)) hide)
     )
@@
       (effects (font (size 1.27 1.27)) (justify right))
     )
-    (property "Footprint" "Diode_SMD:D_SOD-123" (id 2) (at 263.525 144.78 0)
-      (effects (font (size 1.27 1.27)) hide)
-    )
+    (property "Footprint" "Diode_SMD:D_0402_1005Metric" (id 2) (at 263.525 144.78 0)
+      (effects (font (size 1.27 1.27)) hide)
+    )

Commit message: Release v0.1
Other:
- company: (none) -> Polskie Towarzystwo Rakietowe
- title: (none) -> KP-PTR
- moved on the sheet: ANT2, C16, C17, C19, C23, C24, C25, C26, C30, C32, D1, D2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
